File: EE1_project.kicad_pcb (KiCad board)
At the start: 2 copper layers, 50 x 50 mm, 33 parts, among them J1 GUESS RESISTOR 1, J2 GUESS RESISTOR 2, J3 GUESS RESISTOR 3, J4 POWER, Q1 2N7000, Q2 2N7000, SW1 TEST, U1 LM358

Commit message: flip smd and traces to back
Parts:
- C1, C2, C3, C4, R1, R2, R3, R4, R5, R6, R7, R8: moved to B.Cu
Routing:
- added copper zone on B.Cu, net GND
- removed copper zone on F.Cu, net GND
Other:
- board text added: "LOWER THRESHOLD"
- board text added: "TEST HOLD"
- board text added: "UPPER THRESHOLD"
